File: 33.sch (KiCad schematic (older format))
At the start: 77 parts, among them U1 ProMicro

Commit message: breakout 4 unused pins
Parts:
- added J1, J2: Conn_01x02_Female, Connector_JST:JST_EH_B2B-EH-A_1x02_P2.50mm_Vertical, symbol Connector:Conn_01x02_Female
Connections:
- net at U1.1 (TX0/PD3): now also J1.2 (Pin_2)
- net at U1.13 (10/PB6): now also J2.2 (Pin_2)
- net at U1.14 (16/PB2): now also J2.1 (Pin_1)
- net at U1.2 (RX1/PD2): now also J1.1 (Pin_1)
- no-connect marks 5 -> 1
Changed lines of the file:
@@
 Text GLabel 1950 3750 0    50   Input ~ 0
 ROW3
-NoConn ~ 3350 3650
-NoConn ~ 3350 3750
 Wire Wire Line
 	3700 2750 3700 2500
@@
 	3700 2500 3950 2500
 Connection ~ 3950 2500
-NoConn ~ 1950 2650
-NoConn ~ 1950 2750
 NoConn ~ 3350 2650
+$Comp
+L Connector:Conn_01x02_Female J2
+U 1 1 5F899C6B
+P 3550 3650
+F 0 "J2" H 3578 3626 50  0000 L CNN
+F 1 "Conn_01x02_Female" H 3578 3535 50  0000 L CNN
+F 2 "Connector_JST:JST_EH_B2B-EH-A_1x02_P2.50mm_Vertical" H 3550 3650 50  0001 C CNN
+F 3 "~" H 3550 3650 50  0001 C CNN
+	1    3550 3650
+	1    0    0    -1
+$EndComp
+$Comp
+L Connector:Conn_01x02_Female J1
+U 1 1 5F89A905
+P 1750 2750
+F 0 "J1" H 1642 2425 50  0000 C CNN
+F 1 "Conn_01x02_Female" H 1642 2516 50  0000 C CNN
+F 2 "Connector_JST:JST_EH_B2B-EH-A_1x02_P2.50mm_Vertical" H 1750 2750 50  0001 C CNN
+F 3 "~" H 1750 2750 50  0001 C CNN
+	1    1750 2750
+	-1   0    0    1
+$EndComp
 $EndSCHEMATC
